File: eagle/EFM_VCF_4622.brd (EAGLE design)
At the start: 100 x 80 mm, 57 parts, among them IC1 LM13700N, Q1 2N3904, Q10 2N3904, Q11 2N3904, Q12 2N3904, Q13 2N3904, Q2 2N3904, Q3 2N3906, Q4 2N3904, Q5 2N3904, Q6 2N3904, Q7 2N3904, Q8 2N3904, Q9 2N3904, U1 POWER

Commit message: board progress
Parts:
- removed U$1, U$2, U$3: AUDIO-JACK, erthenvar:ERTHENVAR-JACK-90DEG
- added CV1, IN1, OUT: AUDIO-JACK, erthenvar:ERTHENVAR-JACK-90DEG
- moved C12 179.6 mm to (92.7, 24.1)
- moved Q5 156.7 mm to (71.1, 24.1), turned to 270 degrees
- moved C11 147.0 mm to (66.0, 14.0), turned to 90 degrees
- moved CUTOFF 138.8 mm to (80.0, 3.81)
- moved Q10 130.5 mm to (49.5, 50.8), turned to 270 degrees
- moved Q13 126.3 mm to (72.4, 52.1), turned to 270 degrees
- moved RESONANCE 126.1 mm to (63.5, 3.81)
- moved CV1_LEVEL 123.6 mm to (47.0, 3.81)
- moved R3 120.7 mm to (41.9, 76.2)
- moved Q9 115.0 mm to (49.5, 62.2), turned to 270 degrees
- moved C5 113.7 mm to (61.0, 76.2)
- moved R9 112.9 mm to (19.1, 14.0), turned to 90 degrees
- moved R10 112.4 mm to (14.0, 21.6), turned to 180 degrees
- moved R1 112.2 mm to (38.1, 22.9), turned to 90 degrees
- moved Q4 101.1 mm to (25.4, 24.1), turned to 270 degrees
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Connections:
- removed net N$34: IN_2.MP
- net GND: now also CV1.P$1, IN1.P$1, OUT.P$1; no longer U$1.P$1, U$2.P$1, U$3.P$1
- net N$31: now also OUT.P$3; no longer U$3.P$3
- net N$5: now also IN_2.MP
- net N$55: now also CV1.P$2; no longer U$1.P$2
- net N$58: now also IN1.P$3; no longer U$2.P$3
- net N$59: now also CV1.P$3; no longer U$1.P$3

Commit message: parts on the board
Parts:
- removed C12: 10uF, rcl:B45181A
- removed R1: 4k7, rcl:0207/7
- removed R23, R29: 10k, rcl:0207/7
- removed R5: 1k, rcl:0207/7
- added C4: 0.1uF, rcl:C050-025X075
- added R24: 470k, rcl:0207/7
- added R25, R27: 10k, rcl:0207/7
- added R26: 33k, rcl:0207/7
- C5: value 10uF -> 0.1uF; device rcl:B45181A -> rcl:C050-025X075
- C6, C7: device rcl:C025-030X050 -> rcl:C050-025X075
- C8, C9: value 0.1uF -> 10uF; device rcl:C025-030X050 -> rcl:B45181A
- Q1: value 2N3904 -> 2N3906; device transistor-npn:TO92 -> transistor-pnp:TO92
- Q3: value 2N3906 -> 2N3904; device transistor-pnp:TO92 -> transistor-npn:TO92
- R10: value 100k -> 10k
- R11: value 150k -> 4k7
- R14: value 100R -> 1k
- R16: value 10k -> 1k
- R19: value 2k2 -> 1k
- R20: value 33k -> 2k2
- R22: value 470k -> 100R
- R3, R4, R8: value 1k -> 100k
- R6: value 100k -> 150k
- R9: value 100k -> 1k
- moved R22 134.1 mm to (58.4, 14.0), turned to 270 degrees
- moved R13 132.5 mm to (87.6, 48.3)
- moved R14 128.1 mm to (72.4, 47.0), turned to 180 degrees
- moved R16 125.4 mm to (53.3, 61.0), turned to 90 degrees
- moved R15 124.9 mm to (59.7, 49.5), turned to 180 degrees
- moved C6 119.7 mm to (55.9, 61.0), turned to 270 degrees
- moved R17 119.3 mm to (39.4, 73.7), turned to 180 degrees
- moved C7 113.4 mm to (43.2, 61.0), turned to 270 degrees
- moved C9 108.0 mm to (25.4, 54.6), turned to 90 degrees
- moved R8 105.2 mm to (19.1, 14.0), turned to 90 degrees
- moved C8 97.1 mm to (19.1, 71.1), turned to 180 degrees
- moved R4 96.2 mm to (47.0, 14.0), turned to 270 degrees
- moved R7 88.9 mm to (14.0, 21.6), turned to 180 degrees
- moved R11 87.5 mm to (38.1, 22.9), turned to 90 degrees
- moved R6 84.9 mm to (27.9, 31.8), turned to 180 degrees
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- renumbered CV1 to CV_1, CV1_LEVEL to CV1_LEV, IN1_LEVEL to IN1_LEV, IN_2 to IN2, R2 to R21, RESONANCE to Q, U1 to PWR1
Connections:
- removed net N$16: Q3.2, R11.1, R12.1, R6.1, R7.1
- new net N$20: Q1.2, R3.1, R4.1, R6.1, R9.1
- net +12V: now also Q13.1; no longer Q5.1
- net -12V: now also R25.2, R27.2, R6.2; no longer R1.2, R23.2, R29.2
- net GND: now also C8.-, C9.-, Q2.3, R24.2, R26.2, R9.2; no longer C10.-, C3.-, Q4.3, R12.2, R19.2, R22.2
- net N$1: now also R24.1; no longer R22.1
- net N$10: now also C10.+; no longer C11.+
- net N$12: now also C4.1, Q8.3, Q9.1; no longer C6.1, Q11.1, Q13.3
- net N$13: now also C6.1, Q10.3, Q11.1; no longer C7.1, Q7.1, Q9.3
- net N$14: now also C5.2, Q4.3, Q5.1; no longer C8.2, Q10.3, Q8.1
- net N$15: now also C5.1, Q10.1, Q9.3; no longer C8.1, Q11.3, Q9.1
- net N$17: now also C7.1, Q11.3, Q12.1; no longer C9.1, Q2.1, Q7.3
- net N$18: now also C7.2, Q7.1; no longer C9.2, Q1.1
- net N$19: now also Q13.2, R26.1; no longer Q5.2, R20.1
- net N$2: now also R22.2; no longer R14.2
- net N$25: now also C8.+, R12.2, R17.2, R19.2, R20.1; no longer C10.+, R15.2, R18.2, R19.1, R3.2
- net N$26: now also Q12.2, R19.1, R22.1; no longer Q2.2, R14.1, R18.1
- net N$27: now also Q1.1, R11.1; no longer Q3.1, R1.1
- net N$28: now also C11.+, R27.1; no longer C12.+, R29.1
- net N$29: now also C6.2, Q5.3; no longer C7.2, Q8.3
- net N$3: now also Q2.1, R18.2; no longer Q4.1, R17.2
- net N$31: now also C11.-; no longer C12.-
- net N$35: now also C10.-, Q13.3, R25.1; no longer C11.-, Q5.3, R23.1
- net N$38: now also C9.+, R10.1; no longer C3.+, R16.1
- net N$4: now also Q12.3, Q7.3, R18.1; no longer Q1.3, Q2.3, R17.1
- net N$43: now also Q3.1, Q8.1; no longer Q12.1, Q13.1
- net N$44: now also Q3.2, Q8.2, R14.1; no longer Q12.2, Q13.2, R8.1
- net N$46: now also Q4.2, Q9.2, R14.2, R15.1; no longer Q10.2, Q11.2, R5.1, R8.2
- net N$49: now also Q10.2, Q5.2, R15.2, R16.1; no longer Q8.2, Q9.2, R4.1, R5.2
- net N$5: now also R7.2; no longer R10.2
- net N$50: now also Q11.2, R16.2, R17.1; no longer Q7.2, R3.1, R4.2
- net N$53: now also R4.2; no longer R7.2
- net N$56: now also R3.2; no longer R6.2
- net N$57: now also R8.1; no longer R9.1
- net N$6: now also C3.-, R7.1, R8.2; no longer C5.-, R10.1, R9.2
- net N$7: now also C3.+, Q7.2, R12.1; no longer C5.+, Q1.2, R15.1
- net N$8: now also Q1.3, Q2.2, R10.2; no longer Q3.3, Q4.2, R16.2
- net N$9: now also C4.2, Q3.3, Q4.1; no longer C6.2, Q10.1, Q12.3

Commit message: trying routes
Parts:
- moved R21 86.9 mm to (82.5, 69.8)
- moved R14 20.7 mm to (87.6, 61.0)
- moved C4 15.3 mm to (71.1, 43.2), turned to 180 degrees
- moved R18 13.5 mm to (30.5, 66.0)
- moved R15 12.0 mm to (63.5, 61.0)
- moved R6 8.89 mm to (36.8, 31.8), turned to 0 degrees
- moved R19 7.18 mm to (33.0, 73.7), turned to 180 degrees
- moved R17 6.48 mm to (45.7, 74.9)
- moved R16 3.81 mm to (53.3, 64.8)
- moved R9 2.84 mm to (29.2, 39.4)
- moved Q2 1.80 mm to (26.7, 25.4), turned to 180 degrees
- moved Q1 1.27 mm to (31.8, 25.4)
Routing:
- net GND: track 0.00 -> 251.6 mm
- net N$38: track 0.00 -> 218.8 mm
- net N$26: track 0.00 -> 141.6 mm
- net -12V: track 0.00 -> 99.4 mm
- net N$20: track 0.00 -> 82.6 mm
- net N$19: track 0.00 -> 63.9 mm
- net N$35: track 0.00 -> 48.2 mm
- net N$43: track 0.00 -> 44.5 mm
- net N$25: track 0.00 -> 44.1 mm
- net N$44: track 0.00 -> 38.9 mm
- net N$9: track 0.00 -> 33.9 mm
- net N$49: track 0.00 -> 31.5 mm
- net N$46: track 0.00 -> 27.9 mm
- net N$50: track 0.00 -> 23.7 mm
- net N$4: track 0.00 -> 23.7 mm
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
Commit message: routed
Parts:
- C10, C3: device rcl:B45181A -> rcl:B45181B
- C11: device rcl:B45181A -> rcl:B45181C
- R10: device rcl:0207/7 -> rcl:0309/12
- moved R18 22.5 mm to (36.8, 44.5), turned to 180 degrees
- moved C11 9.16 mm to (87.6, 31.8)
- moved R9 6.35 mm to (34.3, 35.6), turned to 180 degrees
- moved R25 5.39 mm to (50.8, 21.6)
- moved Q13 5.08 mm to (66.0, 24.1), turned to 90 degrees
- moved R3 4.58 mm to (76.2, 11.4), turned to 0 degrees
- moved R6 3.81 mm to (40.6, 31.8)
- moved R27 3.59 mm to (50.8, 35.6), turned to 180 degrees
- moved R12 3.59 mm to (30.5, 63.5)
- moved R17 2.84 mm to (43.2, 73.7)
- moved R16 2.84 mm to (52.1, 62.2)
- moved C3 2.84 mm to (16.5, 27.9)
- moved C8 2.54 mm to (19.1, 68.6)
- moved Q3 2.54 mm to (85.1, 55.9)
- moved Q4 2.54 mm to (77.5, 55.9), turned to 0 degrees
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Routing:
- net N$7: track 8.75 -> 55.1 mm, vias 0 -> 2
- net N$58: track 0.00 -> 41.0 mm
- net N$12: track 6.13 -> 46.6 mm, vias 0 -> 4
- net N$3: track 0.00 -> 37.4 mm
- net N$59: track 0.00 -> 34.1 mm
- net N$35: track 48.2 -> 15.8 mm
- net GND: track 251.6 -> 283.0 mm
- net N$28: track 5.61 -> 33.6 mm
- net N$20: track 82.6 -> 59.5 mm
- net N$31: track 0.00 -> 17.6 mm
- net N$13: track 8.45 -> 22.4 mm, vias 0 -> 2
- net N$19: track 63.9 -> 53.6 mm
- net N$8: track 21.9 -> 16.0 mm
- net N$44: track 38.9 -> 44.9 mm
- net N$50: track 23.7 -> 19.3 mm
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
Commit message: fixed connections
Parts:
- R24: device rcl:0207/7 -> rcl:0309/12
- moved R21 29.7 mm to (91.4, 43.2), turned to 270 degrees
- moved R22 12.2 mm to (71.6, 12.7), turned to 180 degrees
- moved R24 9.25 mm to (82.5, 29.2), turned to 270 degrees
- moved R3 6.35 mm to (76.2, 17.8)
- moved R27 5.68 mm to (53.3, 40.6), turned to 90 degrees
- moved IN2 4.02 mm to (7.62, 21.6)
- moved R14 3.81 mm to (83.8, 61.0)
- moved C11 2.84 mm to (90.4, 32.3)
- moved Q13 2.54 mm to (63.5, 24.1)
- moved C9 2.54 mm to (25.4, 52.1)
- moved R12 1.80 mm to (31.8, 62.2)
- moved R11 1.80 mm to (38.1, 22.9)
- moved Q3 1.27 mm to (83.8, 55.9)
- moved Q1 1.27 mm to (31.8, 26.7)
- moved Q2 1.27 mm to (26.7, 26.7)
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Connections:
- removed net N$38: C1.+, C9.+, CUTOFF.3, PWR1.10, PWR1.9, R10.1, R21.2
- net +12V: now also C1.+, C9.+, CUTOFF.3, PWR1.10, PWR1.9, R10.1, R21.2
Routing:
- net +12V: track 6.91 -> 277.7 mm
- net N$38: track 222.6 -> 0.00 mm
- net N$55: track 2.54 -> 73.7 mm
- net GND: track 283.0 -> 335.1 mm
- net N$2: track 12.8 -> 26.0 mm
- net N$43: track 45.7 -> 37.2 mm
- net N$44: track 44.9 -> 36.7 mm
- net N$25: track 47.3 -> 39.3 mm
- net N$19: track 53.6 -> 60.4 mm
- net N$20: track 59.5 -> 52.9 mm
- net N$56: track 7.62 -> 14.0 mm
- net -12V: track 96.6 -> 101.7 mm
- net N$26: track 140.7 -> 136.2 mm
- net N$5: track 6.88 -> 2.54 mm
- net N$46: track 27.3 -> 23.7 mm
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
Commit message: routed
Parts:
- moved Q8 2.54 mm to (85.1, 67.3), turned to 90 degrees
- moved R16 1.27 mm to (52.1, 63.5)
- moved Q4 1.27 mm to (76.2, 55.9)
Routing:
- net N$44: track 36.7 -> 21.9 mm
- net N$43: track 37.2 -> 40.2 mm
- net N$14: track 15.4 -> 13.7 mm
- net N$12: track 46.4 -> 44.8 mm
- net N$49: track 29.2 -> 27.8 mm
- net N$9: track 32.4 -> 33.3 mm
- net N$13: track 22.4 -> 21.5 mm
- net N$26: track 136.2 -> 135.5 mm
- net N$50: track 19.8 -> 20.4 mm

Commit message: will try cut
Parts:
- C11: device rcl:B45181C -> rcl:B45181B
Routing:
- net N$28: track 36.4 -> 38.8 mm
- net N$26: track 135.5 -> 136.8 mm
- net +12V: track 277.4 -> 276.6 mm
Other:
- board size 100 x 80 mm -> 102.1 x 80.8 mm
Changed lines of the file:
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@@
 <layer number="44" name="Drills" color="7" fill="1" visible="no" active="yes"/>
 <layer number="45" name="Holes" color="7" fill="1" visible="no" active="yes"/>
-<layer number="46" name="Milling" color="3" fill="1" visible="no" active="yes"/>
+<layer number="46" name="Milling" color="3" fill="1" visible="yes" active="yes"/>
 <layer number="47" name="Measures" color="7" fill="1" visible="no" active="yes"/>
 <layer number="48" name="Document" color="7" fill="1" visible="yes" active="yes"/>
@@
 <wire x1="100" y1="80" x2="0" y2="80" width="0" layer="20"/>
 <wire x1="0" y1="80" x2="0" y2="0" width="0" layer="20"/>
+<wire x1="-0.508" y1="-0.762" x2="0" y2="63.5" width="1.6764" layer="46"/>
+<wire x1="0" y1="63.5" x2="26.67" y2="80.01" width="1.6764" layer="46"/>
+<wire x1="26.67" y1="80.01" x2="53.34" y2="80.01" width="1.6764" layer="46"/>
+<wire x1="53.34" y1="80.01" x2="97.79" y2="77.47" width="1.6764" layer="46"/>
+<wire x1="97.79" y1="77.47" x2="97.79" y2="21.59" width="1.6764" layer="46"/>
+<wire x1="97.79" y1="21.59" x2="101.6" y2="17.78" width="1.6764" layer="46"/>
+<wire x1="101.6" y1="17.78" x2="101.6" y2="1.27" width="1.6764" layer="46"/>
+<wire x1="101.6" y1="1.27" x2="98.552" y2="-0.762" width="1.6764" layer="46"/>
+<wire x1="98.552" y1="-0.762" x2="-0.508" y2="-0.762" width="1.6764" layer="46"/>
 </plain>
 <attributes>
@@
 <element name="C8" library="rcl" package="B45181A" value="10uF" x="19.05" y="68.58" rot="R180"/>
 <element name="C10" library="rcl" package="B45181B" value="10uF" x="64.77" y="16.51" rot="R90"/>
-<element name="C11" library="rcl" package="B45181C" value="10uF" x="90.424" y="32.258"/>
+<element name="C11" library="rcl" package="B45181B" value="10uF" x="90.424" y="32.258"/>
 <element name="C2" library="rcl" package="B45181A" value="10uF" x="19.05" y="58.42" rot="R90"/>
 <element name="C9" library="rcl" package="B45181A" value="10uF" x="25.4" y="52.07" rot="R90"/>
@@
 <wire x1="35.56" y1="57.785" x2="35.433" y2="57.7215" width="0.8128" layer="16"/>
 <wire x1="16.51" y1="30.48" x2="16.51" y2="40.64" width="0.8128" layer="16"/>
-<wire x1="16.51" y1="40.64" x2="29.21" y2="46.99" width="0.8128" layer="16"/>
-<via x="29.21" y="46.99" extent="1-16" drill="0.6" diameter="0.8128" shape="square"/>
-<wire x1="29.21" y1="46.99" x2="36.83" y2="46.99" width="0.8128" layer="1"/>
+<wire x1="16.51" y1="40.64" x2="31.75" y2="46.99" width="0.8128" layer="16"/>
+<via x="31.75" y="46.99" extent="1-16" drill="0.6" diameter="0.8128" shape="square"/>
+<wire x1="31.75" y1="46.99" x2="36.83" y2="46.99" width="0.8128" layer="1"/>
 <wire x1="36.83" y1="46.99" x2="39.37" y2="49.53" width="0.8128" layer="1"/>
 <wire x1="39.37" y1="49.53" x2="39.37" y2="58.42" width="0.8128" layer="1"/>
@@
 <contactref element="Q2" pad="1"/>
 <contactref element="R18" pad="2"/>
-<wire x1="33.02" y1="44.45" x2="29.21" y2="44.45" width="0.8128" layer="16"/>
-<wire x1="29.21" y1="44.45" x2="18.288" y2="39.624" width="0.8128" layer="16"/>
+<wire x1="33.02" y1="44.45" x2="18.288" y2="39.624" width="0.8128" layer="16"/>
 <wire x1="18.288" y1="39.624" x2="18.288" y2="33.274" width="0.8128" layer="16"/>
 <wire x1="18.288" y1="33.274" x2="21.59" y2="27.94" width="0.8128" layer="16"/>
@@
 <wire x1="35.56" y1="69.215" x2="36.195" y2="71.12" width="0.8128" layer="16"/>
 <wire x1="36.195" y1="71.12" x2="36.195" y2="71.4375" width="0.6604" layer="16"/>
-<wire x1="88.3285" y1="30.353" x2="81.5975" y2="29.21" width="0.8128" layer="16"/>
-<wire x1="88.3285" y1="41.8465" x2="88.3285" y2="30.353" width="0.8128" layer="16"/>
+<wire x1="89.5985" y1="35.433" x2="89.4715" y2="30.226" width="0.8128" layer="16"/>
+<wire x1="88.3285" y1="41.8465" x2="89.5985" y2="35.433" width="0.8128" layer="16"/>
 <wire x1="93.5355" y1="45.0215" x2="88.3285" y2="41.8465" width="0.8128" layer="16"/>
 <wire x1="93.5355" y1="63.4365" x2="93.5355" y2="45.0215" width="0.8128" layer="16"/>
@@
 <wire x1="40.3225" y1="71.12" x2="44.45" y2="75.7555" width="0.8128" layer="16"/>
 <wire x1="40.3225" y1="71.12" x2="36.195" y2="71.12" width="0.8128" layer="16"/>
-<wire x1="81.5975" y1="29.21" x2="76.2" y2="27.178" width="0.8128" layer="16"/>
+<wire x1="89.4715" y1="30.226" x2="76.2" y2="27.178" width="0.8128" layer="16"/>
 <wire x1="76.2" y1="27.178" x2="76.2" y2="13.462" width="0.8128" layer="16"/>
 <wire x1="76.2" y1="13.462" x2="75.438" y2="12.7" width="0.8128" layer="16"/>
@@
 <wire x1="58.42" y1="34.29" x2="59.69" y2="33.528" width="0.8128" layer="16"/>
 <wire x1="59.69" y1="33.528" x2="81.28" y2="33.528" width="0.8128" layer="16"/>
-<wire x1="81.28" y1="33.528" x2="85.344" y2="32.258" width="0.8128" layer="16"/>
+<wire x1="81.28" y1="33.528" x2="87.884" y2="32.258" width="0.8128" layer="16"/>
 </signal>
 <signal name="N$31">
 <contactref element="C11" pad="-"/>
 <contactref element="OUT" pad="P$3"/>
-<wire x1="95.504" y1="32.258" x2="95.25" y2="19.05" width="0.8128" layer="16"/>
+<wire x1="92.964" y1="32.258" x2="95.25" y2="19.05" width="0.8128" layer="16"/>
 <wire x1="95.25" y1="19.05" x2="95.25" y2="16.89" width="0.8128" layer="16"/>
 <wire x1="95.25" y1="16.89" x2="94.06" y2="15.7" width="0.8128" layer="16"/>
@@
 <wire x1="74.422" y1="20.574" x2="69.596" y2="25.4" width="0.8128" layer="16"/>
 <wire x1="69.596" y1="25.4" x2="63.5" y2="25.4" width="0.8128" layer="16"/>
-<wire x1="91.44" y1="39.37" x2="91.44" y2="27.94" width="0.8128" layer="16"/>
-<wire x1="91.44" y1="27.94" x2="86.36" y2="26.67" width="0.8128" layer="16"/>
+<wire x1="91.44" y1="39.37" x2="91.44" y2="29.21" width="0.8128" layer="16"/>
+<wire x1="91.44" y1="29.21" x2="86.36" y2="26.67" width="0.8128" layer="16"/>
 <wire x1="81.28" y1="26.67" x2="80.01" y2="24.13" width="0.8128" layer="16"/>
 <wire x1="80.01" y1="24.13" x2="80.01" y2="21.59" width="0.8128" layer="16"/>

Commit message: ready to cut
Parts:
- moved R22 6.35 mm to (69.8, 18.8), turned to 270 degrees
- moved C4 6.14 mm to (74.2, 48.5), turned to 0 degrees
- moved R24 3.30 mm to (82.5, 32.5)
- moved R26 3.07 mm to (40.6, 36.6)
- moved R13 2.84 mm to (88.9, 52.1)
- moved R16 2.84 mm to (50.8, 61.0), turned to 180 degrees
- moved R9 2.84 mm to (35.6, 33.0)
- moved C8 2.84 mm to (20.3, 66.0)
- moved C11 2.54 mm to (90.4, 34.8)
- moved R6 2.54 mm to (40.6, 29.2)
- moved R19 2.34 mm to (31.5, 71.9)
- moved R17 1.78 mm to (43.2, 71.9)
- moved C5 1.27 mm to (69.8, 59.7)
- moved R27 1.27 mm to (53.3, 39.4)
- moved Q10 1.27 mm to (62.2, 66.0)
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Routing:
- net +12V: track 276.6 -> 250.7 mm
- net N$9: track 33.3 -> 52.3 mm
- net N$26: track 136.8 -> 125.7 mm
- net N$58: track 42.0 -> 34.6 mm
- net N$19: track 60.4 -> 53.0 mm
- net GND: track 335.1 -> 329.2 mm
- net -12V: track 101.7 -> 97.5 mm
- net N$43: track 40.2 -> 36.1 mm
- net N$25: track 39.7 -> 36.3 mm
- net N$50: track 20.4 -> 17.8 mm
- net N$31: track 17.2 -> 19.8 mm
- net N$44: track 21.9 -> 19.4 mm
- net N$7: track 53.1 -> 51.3 mm
- net N$20: track 52.9 -> 51.1 mm
- net N$49: track 27.8 -> 26.1 mm
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Other:
- board size 102.1 x 80.8 mm -> 101.6 x 80.8 mm
